File: 286TowerOfSomething/compagne-supernova/compagne-supernova.kicad_pcb (KiCad board)
At the start: 2 copper layers, 38 parts, among them J1 Bus_ISA_8bit, J2 DE9, J3 DE9, J4 Mini-DIN-6, SW1 SW_DIP_x04, U1 16550, U2 GD75232N, U3 74HCU04, U4 74LS138, U5 74LS138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

Commit message: Doing some work on the compagne-supernova layout
Parts:
- moved C10 24.9 mm to (126.7, 99.4), turned to 180 degrees
- moved C9 13.9 mm to (116.0, 99.4), turned to 180 degrees
Connections:
- U8 pad 6: /PS2 to Serial/RX -> /RX
- U8 pad 7: /PS2 to Serial/~{RTS} -> /~{RTS}
Routing:
- net /RX: track 0.00 -> 70.1 mm, vias 0 -> 3
- net Net-(U6-SIN): track 0.00 -> 65.3 mm, vias 0 -> 1
- net Net-(U6-SOUT): track 0.00 -> 62.7 mm, vias 0 -> 1
- net /~{RTS}: track 0.00 -> 55.4 mm, vias 0 -> 3
- net Net-(U6-~{RTS}): track 0.00 -> 45.7 mm, vias 0 -> 1
- net Net-(U1-SOUT): track 0.00 -> 40.6 mm, vias 0 -> 1
- net Net-(U6-~{DSR}): track 0.00 -> 38.1 mm, vias 0 -> 1
- net Net-(U6-~{DCD}): track 0.00 -> 38.0 mm, vias 0 -> 1
- net Net-(U1-~{DCD}): track 0.00 -> 37.8 mm, vias 0 -> 1
- net Net-(U6-~{DTR}): track 0.00 -> 35.6 mm, vias 0 -> 1
- net Net-(U1-~{DTR}): track 0.00 -> 31.1 mm, vias 0 -> 1
- net Net-(U6-~{CTS}): track 0.00 -> 30.5 mm, vias 0 -> 1
- net Net-(U1-~{DSR}): track 0.00 -> 30.2 mm, vias 0 -> 1
- net /~{0x2F8}: track 0.00 -> 23.3 mm
- net /~{0x2E8}: track 0.00 -> 23.3 mm
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