File: 286TowerOfSomething/dmp-go-away/ide.kicad_sch (KiCad schematic)
At the start: 0 parts

Commit message: Adding work done on 386 card, coming along nicely
Parts:
- added C23, C24: 100n, symbol Device:C
- added J2: Conn_02x20_Odd_Even, symbol Connector_Generic:Conn_02x20_Odd_Even
- added U7, U8: 74LS245, symbol 74xx:74LS245
Connections:
- new net: J2.18 (Pin_18), U8.11 (B7)
- new net: J2.16 (Pin_16), U8.12 (B6)
- new net: J2.14 (Pin_14), U8.13 (B5)
- new net: J2.12 (Pin_12), U8.14 (B4)
- new net: J2.10 (Pin_10), U8.15 (B3)
- new net: J2.8 (Pin_8), U8.16 (B2)
- new net: J2.6 (Pin_6), U8.17 (B1)
- new net: J2.4 (Pin_4), U8.18 (B0)
- new net: J2.3 (Pin_3), U7.11 (B7)
- new net: J2.5 (Pin_5), U7.12 (B6)
- new net: J2.7 (Pin_7), U7.13 (B5)
- new net: J2.9 (Pin_9), U7.14 (B4)
- new net: J2.11 (Pin_11), U7.15 (B3)
- new net: J2.13 (Pin_13), U7.16 (B2)
- new net: J2.15 (Pin_15), U7.17 (B1)
- new net: J2.17 (Pin_17), U7.18 (B0)
- new net +5V: C23.1, C24.1, U7.20 (VCC), U8.20 (VCC)
- new net GND: C23.2, C24.2, J2.19 (Pin_19), J2.2 (Pin_2), J2.22 (Pin_22), J2.24 (Pin_24), J2.26 (Pin_26), J2.30 (Pin_30), J2.40 (Pin_40), U7.10 (GND), U8.10 (GND)
- new net IDEEN: U7.19 (CE), U8.19 (CE)
- new net IDELED: J2.39 (Pin_39)
- new net IRQ14: J2.31 (Pin_31)
- new net SA0: J2.35 (Pin_35)
- new net SA1: J2.33 (Pin_33)
- new net SA2: J2.36 (Pin_36)
- new net SD0: U7.2 (A0)
- new net SD1: U7.3 (A1)
- new net SD10: U8.4 (A2)
- new net SD11: U8.5 (A3)
- new net SD12: U8.6 (A4)
- new net SD13: U8.7 (A5)
- new net SD14: U8.8 (A6)
- new net SD15: U8.9 (A7)
- new net SD2: U7.4 (A2)
- new net SD3: U7.5 (A3)
- new net SD4: U7.6 (A4)
- new net SD5: U7.7 (A5)
- new net SD6: U7.8 (A6)
- new net SD7: U7.9 (A7)
- new net SD8: U8.2 (A0)
- new net SD9: U8.3 (A1)
- new net ~{IDECS0}: J2.37 (Pin_37)
- new net ~{IDECS1}: J2.38 (Pin_38)
- new net ~{IOCS16}: J2.32 (Pin_32)
- new net ~{IOR}: J2.25 (Pin_25), U7.1 (A->B), U8.1 (A->B)
- new net ~{IOW}: J2.23 (Pin_23)
- new net ~{RESETL}: J2.1 (Pin_1)
- no-connect marks 0 -> 6

Commit message: Added footprints and started figuring out layout for dmp-go-away
Parts:
- C23, C24: footprint (none) -> Capacitor_SMD:C_0603_1608Metric_Pad1.08x0.95mm_HandSolder
- J2: footprint (none) -> Connector_IDC:IDC-Header_2x20_P2.54mm_Vertical
- U7, U8: footprint (none) -> Package_SO:SSOP-20_5.3x7.2mm_P0.65mm
Changed lines of the file:
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@@
 			)
 		)
-		(property "Footprint" ""
+		(property "Footprint" "Capacitor_SMD:C_0603_1608Metric_Pad1.08x0.95mm_HandSolder"
 			(at 242.2652 54.61 0)
 			(effects
@@
 			)
 		)
-		(property "Footprint" ""
+		(property "Footprint" "Package_SO:SSOP-20_5.3x7.2mm_P0.65mm"
 			(at 127 152.4 0)
 			(effects
@@
 			)
 		)
-		(property "Footprint" ""
+		(property "Footprint" "Package_SO:SSOP-20_5.3x7.2mm_P0.65mm"
 			(at 127 76.2 0)
 			(effects
@@
 			)
 		)
-		(property "Footprint" ""
+		(property "Footprint" "Capacitor_SMD:C_0603_1608Metric_Pad1.08x0.95mm_HandSolder"
 			(at 229.5652 54.61 0)
 			(effects
@@
 			)
 		)
-		(property "Footprint" ""
+		(property "Footprint" "Connector_IDC:IDC-Header_2x20_P2.54mm_Vertical"
 			(at 190.5 113.03 0)
 			(effects
