File: 286TowerOfSomething/dmp-go-away/ram.kicad_sch (KiCad schematic)
At the start: 34 parts, among them U1 M6117C, U2 M5M416160CJ, U3 M5M416160CJ, U4 M5M416160CJ, U5 M5M416160CJ

Commit message: Added footprints and started figuring out layout for dmp-go-away
Parts:
- U1: footprint (none) -> Package_QFP:PQFP-208_28x28mm_P0.5mm
- U2, U3, U4, U5: footprint (none) -> pc-parts:SOJ-42
Changed lines of the file:
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@@
 			)
 		)
-		(property "Footprint" ""
+		(property "Footprint" "Package_QFP:PQFP-208_28x28mm_P0.5mm"
 			(at 88.9 102.87 0)
 			(effects
@@
 			)
 		)
-		(property "Footprint" ""
+		(property "Footprint" "pc-parts:SOJ-42"
 			(at 203.2 166.37 0)
 			(effects
@@
 			)
 		)
-		(property "Footprint" ""
+		(property "Footprint" "pc-parts:SOJ-42"
 			(at 152.4 90.17 0)
 			(effects
@@
 			)
 		)
-		(property "Footprint" ""
+		(property "Footprint" "pc-parts:SOJ-42"
 			(at 152.4 166.37 0)
 			(effects
@@
 			)
 		)
-		(property "Footprint" ""
+		(property "Footprint" "pc-parts:SOJ-42"
 			(at 203.2 90.17 0)
 			(effects
