File: 286TowerOfSomething/dmp-go-away/dmp-go-away.kicad_pcb (KiCad board)
At the start: 2 copper layers, 91 parts, among them J1 Bus_ISA_16bit, J2 Conn_02x20_Odd_Even, J3 Keyboard, J4 Mouse, Q1 MMBT3904, U1 M6117C, U2 M5M416160CJ, U3 M5M416160CJ, U4 M5M416160CJ, U5 M5M416160CJ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

Commit message: Adding bracket to dmp-go-away
Parts:
- added BRACKET1: ~, pc-parts:PC_BRACKET_ISA_KEYSTONE_9202_Rev1, F.Cu at (241.3, 133.3)
- moved C1 191.8 mm to (13.4, -30.4)
- moved C18 191.8 mm to (85.2, -121.7)
- moved C19 191.8 mm to (85.2, -119.2)
- moved C2 191.8 mm to (13.4, -27.8)
- moved C20 191.8 mm to (85.2, -116.6)
- moved C21 191.8 mm to (85.2, -114.1)
- moved C22 191.8 mm to (85.2, -111.6)
- moved C3 191.8 mm to (13.4, -25.3)
- moved C32 191.8 mm to (22.4, 24.4)
- moved C33 191.8 mm to (22.4, 26.9)
- moved C4 191.8 mm to (13.4, -22.8)
- moved C5 191.8 mm to (107.7, -138.5)
- moved D1 191.8 mm to (114.6, -139.6)
- moved J2 191.8 mm to (46.2, -173.3)
- moved JP2 191.8 mm to (67.6, -101.9)
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Other:
- board outline added: 242.4 x 106.7 mm
