File: 286TowerOfSomething/ethermaker/ethermaker.kicad_pcb (KiCad board)
At the start: 2 copper layers, 29 parts, among them J1 Bus_ISA_16bit, J2 RJ45_Hanrun_HR911105A_Horizon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, U1 CS8900A, U2 GAL16V8, U3 93C46A, U4 SST39SF010, U5 74LS245, Y1 20.0 MHz

Commit message: Work on ethermaker layout
Parts:
- moved C12 116.5 mm to (227.0, 78.7)
- moved C13 116.5 mm to (227.0, 85.6)
- moved C14 116.5 mm to (227.0, 92.4)
- moved JP1 42.1 mm to (118.1, 82.5), turned to 180 degrees
- moved R4 28.7 mm to (187.3, 73.7)
- moved J1 25.2 mm to (171.4, 123.2)
- moved C2 24.0 mm to (142.2, 70.5)
- moved C6 23.5 mm to (128.5, 87.6)
- moved C7 23.0 mm to (128.5, 80.6)
- moved U1 22.9 mm to (139.7, 82.5)
- moved Y1 22.9 mm to (132.9, 69.3)
- moved C3 22.8 mm to (145.4, 70.5)
- moved C9 22.8 mm to (118.1, 69.2)
- moved C4 22.6 mm to (150.5, 79.4)
- moved C5 22.5 mm to (150.5, 86.0)
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Routing:
- net /DRQ7: track 0.00 -> 119.5 mm, vias 0 -> 1
- net /~{DACK7}: track 0.00 -> 116.3 mm, vias 0 -> 1
- net /DRQ6: track 0.00 -> 113.2 mm, vias 0 -> 1
- net /D15: track 0.00 -> 110.4 mm
- net /~{DACK6}: track 0.00 -> 110.1 mm, vias 0 -> 1
- net /D14: track 0.00 -> 107.6 mm
- net /DRQ5: track 0.00 -> 107.0 mm, vias 0 -> 1
- net /D13: track 0.00 -> 104.9 mm
- net /~{DACK5}: track 0.00 -> 103.9 mm, vias 0 -> 1
- net /D11: track 0.00 -> 102.7 mm
- net /D12: track 0.00 -> 102.1 mm
- net /D10: track 0.00 -> 99.9 mm
- net /D9: track 0.00 -> 96.3 mm
- net /D8: track 0.00 -> 94.3 mm
- net /IRQ12: track 0.00 -> 79.7 mm, vias 0 -> 1
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- added copper zone on B.Cu, net GND
- added copper zone on F.Cu, net GND
Other:
- board outline added: 161.1 x 90.2 mm

Commit message: I think that's an Ethernet carD
Parts:
- moved C14 183.2 mm to (44.5, 108.2), turned to 180 degrees
- moved C10 129.4 mm to (189.2, 103.9), turned to -90 degrees
- moved C12 119.8 mm to (107.4, 70.4), turned to 90 degrees
- moved U5 103.1 mm to (186.7, 100.1), turned to -90 degrees
- moved U4 95.3 mm to (148.6, 96.5), turned to 90 degrees
- moved C8 88.8 mm to (148.6, 78.0), turned to 90 degrees
- moved C13 61.9 mm to (171.4, 113.0), turned to 180 degrees
- moved C11 55.2 mm to (87.6, 111.0), turned to -90 degrees
- moved U2 50.6 mm to (87.6, 100.1), turned to -90 degrees
- moved JP1 45.6 mm to (82.5, 111.0), turned to -90 degrees
- moved C2 43.2 mm to (99.1, 70.5)
- moved C4 43.2 mm to (107.3, 79.4)
- moved C5 43.2 mm to (107.3, 86.0)
- moved C6 43.2 mm to (85.3, 87.6)
- moved C7 43.2 mm to (85.3, 80.6)
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Connections:
- J2 pad 12: Net-(J2-Pad12) -> +5V
- J2 pad 9: Net-(J2-Pad12) -> +5V
Routing:
- net +5V: track 74.4 -> 388.2 mm, vias 0 -> 6
- net /ROM_CS: track 24.6 -> 121.6 mm, vias 0 -> 1
- net /A10: track 43.8 -> 131.0 mm, vias 0 -> 3
- net /RESET: track 64.1 -> 149.9 mm, vias 1 -> 3
- net /A11: track 41.9 -> 126.3 mm, vias 0 -> 3
- net /A12: track 41.2 -> 124.6 mm, vias 0 -> 3
- net /A0: track 63.4 -> 146.7 mm, vias 0 -> 3
- net /A1: track 61.5 -> 143.1 mm, vias 0 -> 3
- net /A2: track 59.5 -> 137.6 mm, vias 0 -> 3
- net /A9: track 45.8 -> 123.8 mm, vias 0 -> 3
- net /A3: track 57.6 -> 131.8 mm, vias 0 -> 3
- net /A8: track 47.8 -> 121.9 mm, vias 0 -> 3
- net /A13: track 45.0 -> 117.9 mm, vias 0 -> 3
- net /A7: track 49.7 -> 121.9 mm, vias 0 -> 3
- net /A6: track 51.7 -> 123.6 mm, vias 0 -> 3
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