File: 286TowerOfSomething/dont-look-backplane-in-anger/dont-look-backplane-in-anger.kicad_pcb (KiCad board)
At the start: 2 copper layers, 7 parts, among them J1 Bus_ISA_16bit, J2 Bus_ISA_16bit, J3 Bus_ISA_16bit, J4 Bus_ISA_16bit, J5 Bus_ISA_16bit, J6 Bus_ISA_16bit, J7 Bus_ISA_16bit

Commit message: Adding an eighth slot to the backplane
Parts:
- added J8: Bus_ISA_16bit, pc-parts:645169-3, F.Cu at (203.2, 92.7)
Routing:
- net /D5: track 128.2 -> 149.6 mm
- net /D2: track 128.2 -> 149.6 mm
- net /A18: track 128.2 -> 149.6 mm
- net /A13: track 128.2 -> 149.6 mm
- net -12V: track 128.2 -> 149.6 mm
- net /MASTER: track 128.2 -> 149.6 mm
- net /LA23: track 128.2 -> 149.6 mm
- net /LA20: track 128.2 -> 149.6 mm
- net /LA17: track 128.2 -> 149.6 mm
- net /IORDY: track 128.2 -> 149.6 mm
- net /DRQ6: track 128.2 -> 149.6 mm
- net /D9: track 128.2 -> 149.6 mm
- net /D6: track 128.2 -> 149.6 mm
- net /D4: track 128.2 -> 149.6 mm
- net /D13: track 128.2 -> 149.6 mm
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
Commit message: Cleaned up schematic, broke layout
Connections:
- J5 pad 11: /~{MEMWR} -> /Sheet 2/~{MEMWR}
- J5 pad 12: /~{MEMRD} -> /Sheet 2/~{MEMRD}
- J5 pad 13: /~{IOW} -> /Sheet 2/~{IOW}
- J5 pad 14: /~{IOR} -> /Sheet 2/~{IOR}
- J5 pad 15: /~{DACK3} -> /Sheet 2/~{DACK3}
- J5 pad 16: /DRQ3 -> /Sheet 2/DRQ3
- J5 pad 17: /~{DACK1} -> /Sheet 2/~{DACK1}
- J5 pad 18: /DRQ1 -> /Sheet 2/DRQ1
- J5 pad 19: /~{REFRESH} -> /Sheet 2/~{REFRESH}
- J5 pad 2: /RESET -> /Sheet 2/RESET
- J5 pad 20: /CLK -> /Sheet 2/CLK
- J5 pad 21: /IRQ7 -> /Sheet 2/IRQ7
- J5 pad 22: /IRQ6 -> /Sheet 2/IRQ6
- J5 pad 23: /IRQ5 -> /Sheet 2/IRQ5
- J5 pad 24: /IRQ4 -> /Sheet 2/IRQ4
- J5 pad 25: /IRQ3 -> /Sheet 2/IRQ3
- J5 pad 26: /~{DACK2} -> /Sheet 2/~{DACK2}
- J5 pad 27: /TC -> /Sheet 2/TC
- J5 pad 28: /ALE -> /Sheet 2/ALE
- J5 pad 30: /OSC -> /Sheet 2/OSC
- J5 pad 32: /IO -> /Sheet 2/IO
- J5 pad 33: /D7 -> /Sheet 2/D7
- J5 pad 34: /D6 -> /Sheet 2/D6
- J5 pad 35: /D5 -> /Sheet 2/D5
- J5 pad 36: /D4 -> /Sheet 2/D4
- J5 pad 37: /D3 -> /Sheet 2/D3
- J5 pad 38: /D2 -> /Sheet 2/D2
- J5 pad 39: /D1 -> /Sheet 2/D1
- J5 pad 4: /IRQ2 -> /Sheet 2/IRQ2
- J5 pad 40: /D0 -> /Sheet 2/D0
- J5 pad 41: /IORDY -> /Sheet 2/IORDY
- J5 pad 42: /AEN -> /Sheet 2/AEN
- J5 pad 43: /A19 -> /Sheet 2/A19
- J5 pad 44: /A18 -> /Sheet 2/A18
- J5 pad 45: /A17 -> /Sheet 2/A17
- J5 pad 46: /A16 -> /Sheet 2/A16
- J5 pad 47: /A15 -> /Sheet 2/A15
- J5 pad 48: /A14 -> /Sheet 2/A14
- J5 pad 49: /A13 -> /Sheet 2/A13
- J5 pad 50: /A12 -> /Sheet 2/A12
- J5 pad 51: /A11 -> /Sheet 2/A11
- J5 pad 52: /A10 -> /Sheet 2/A10
- J5 pad 53: /A9 -> /Sheet 2/A9
- J5 pad 54: /A8 -> /Sheet 2/A8
- J5 pad 55: /A7 -> /Sheet 2/A7
- J5 pad 56: /A6 -> /Sheet 2/A6
- J5 pad 57: /A5 -> /Sheet 2/A5
- J5 pad 58: /A4 -> /Sheet 2/A4
- J5 pad 59: /A3 -> /Sheet 2/A3
- J5 pad 6: /DRQ2 -> /Sheet 2/DRQ2
- J5 pad 60: /A2 -> /Sheet 2/A2
- J5 pad 61: /A1 -> /Sheet 2/A1
- J5 pad 62: /A0 -> /Sheet 2/A0
- J5 pad 63: /~{MEMCS16} -> /Sheet 2/~{MEMCS16}
- J5 pad 64: /~{IOCS16} -> /Sheet 2/~{IOCS16}
- J5 pad 65: /IRQ10 -> /Sheet 2/IRQ10
- J5 pad 66: /IRQ11 -> /Sheet 2/IRQ11
- J5 pad 67: /IRQ12 -> /Sheet 2/IRQ12
- J5 pad 68: /IRQ15 -> /Sheet 2/IRQ15
- J5 pad 69: /IRQ14 -> /Sheet 2/IRQ14
- J5 pad 70: /~{DACK0} -> /Sheet 2/~{DACK0}
- J5 pad 71: /DRQ0 -> /Sheet 2/DRQ0
- J5 pad 72: /~{DACK5} -> /Sheet 2/~{DACK5}
- J5 pad 73: /DRQ5 -> /Sheet 2/DRQ5
- J5 pad 74: /~{DACK6} -> /Sheet 2/~{DACK6}
- J5 pad 75: /DRQ6 -> /Sheet 2/DRQ6
- J5 pad 76: /~{DACK7} -> /Sheet 2/~{DACK7}
- J5 pad 77: /DRQ7 -> /Sheet 2/DRQ7
- J5 pad 79: /MASTER -> /Sheet 2/MASTER
- J5 pad 81: /SBHE -> /Sheet 2/SBHE
- J5 pad 82: /LA23 -> /Sheet 2/LA23
- J5 pad 83: /LA22 -> /Sheet 2/LA22
- J5 pad 84: /LA21 -> /Sheet 2/LA21
- J5 pad 85: /LA20 -> /Sheet 2/LA20
- J5 pad 86: /LA19 -> /Sheet 2/LA19
- J5 pad 87: /LA18 -> /Sheet 2/LA18
- J5 pad 88: /LA17 -> /Sheet 2/LA17
- J5 pad 89: /~{MEMR} -> /Sheet 2/~{MEMR}
- J5 pad 90: /~{MEMW} -> /Sheet 2/~{MEMW}
- J5 pad 91: /D8 -> /Sheet 2/D8
- J5 pad 92: /D9 -> /Sheet 2/D9
- J5 pad 93: /D10 -> /Sheet 2/D10
- J5 pad 94: /D11 -> /Sheet 2/D11
- J5 pad 95: /D12 -> /Sheet 2/D12
- J5 pad 96: /D13 -> /Sheet 2/D13
- J5 pad 97: /D14 -> /Sheet 2/D14
- J5 pad 98: /D15 -> /Sheet 2/D15
- J6 pad 11: /~{MEMWR} -> /Sheet 2/~{MEMWR}
- J6 pad 12: /~{MEMRD} -> /Sheet 2/~{MEMRD}
- J6 pad 13: /~{IOW} -> /Sheet 2/~{IOW}
- J6 pad 14: /~{IOR} -> /Sheet 2/~{IOR}
- J6 pad 15: /~{DACK3} -> /Sheet 2/~{DACK3}
- J6 pad 16: /DRQ3 -> /Sheet 2/DRQ3
- J6 pad 17: /~{DACK1} -> /Sheet 2/~{DACK1}
- J6 pad 18: /DRQ1 -> /Sheet 2/DRQ1
- J6 pad 19: /~{REFRESH} -> /Sheet 2/~{REFRESH}
- J6 pad 2: /RESET -> /Sheet 2/RESET
- J6 pad 20: /CLK -> /Sheet 2/CLK
- J6 pad 21: /IRQ7 -> /Sheet 2/IRQ7
- J6 pad 22: /IRQ6 -> /Sheet 2/IRQ6
- J6 pad 23: /IRQ5 -> /Sheet 2/IRQ5
- J6 pad 24: /IRQ4 -> /Sheet 2/IRQ4
- J6 pad 25: /IRQ3 -> /Sheet 2/IRQ3
- J6 pad 26: /~{DACK2} -> /Sheet 2/~{DACK2}
- J6 pad 27: /TC -> /Sheet 2/TC
- J6 pad 28: /ALE -> /Sheet 2/ALE
- J6 pad 30: /OSC -> /Sheet 2/OSC
- J6 pad 32: /IO -> /Sheet 2/IO
- J6 pad 33: /D7 -> /Sheet 2/D7
- J6 pad 34: /D6 -> /Sheet 2/D6
- J6 pad 35: /D5 -> /Sheet 2/D5
- J6 pad 36: /D4 -> /Sheet 2/D4
- J6 pad 37: /D3 -> /Sheet 2/D3
- J6 pad 38: /D2 -> /Sheet 2/D2
- J6 pad 39: /D1 -> /Sheet 2/D1
- J6 pad 4: /IRQ2 -> /Sheet 2/IRQ2
- J6 pad 40: /D0 -> /Sheet 2/D0
- J6 pad 41: /IORDY -> /Sheet 2/IORDY
- J6 pad 42: /AEN -> /Sheet 2/AEN
- J6 pad 43: /A19 -> /Sheet 2/A19
- J6 pad 44: /A18 -> /Sheet 2/A18
- J6 pad 45: /A17 -> /Sheet 2/A17
- J6 pad 46: /A16 -> /Sheet 2/A16
- J6 pad 47: /A15 -> /Sheet 2/A15
- J6 pad 48: /A14 -> /Sheet 2/A14
- J6 pad 49: /A13 -> /Sheet 2/A13
- J6 pad 50: /A12 -> /Sheet 2/A12
- J6 pad 51: /A11 -> /Sheet 2/A11
- J6 pad 52: /A10 -> /Sheet 2/A10
- J6 pad 53: /A9 -> /Sheet 2/A9
- J6 pad 54: /A8 -> /Sheet 2/A8
- J6 pad 55: /A7 -> /Sheet 2/A7
- J6 pad 56: /A6 -> /Sheet 2/A6
- J6 pad 57: /A5 -> /Sheet 2/A5
- J6 pad 58: /A4 -> /Sheet 2/A4
- J6 pad 59: /A3 -> /Sheet 2/A3
- J6 pad 6: /DRQ2 -> /Sheet 2/DRQ2
- J6 pad 60: /A2 -> /Sheet 2/A2
- J6 pad 61: /A1 -> /Sheet 2/A1
- J6 pad 62: /A0 -> /Sheet 2/A0
- J6 pad 63: /~{MEMCS16} -> /Sheet 2/~{MEMCS16}
- J6 pad 64: /~{IOCS16} -> /Sheet 2/~{IOCS16}
- J6 pad 65: /IRQ10 -> /Sheet 2/IRQ10
- J6 pad 66: /IRQ11 -> /Sheet 2/IRQ11
- J6 pad 67: /IRQ12 -> /Sheet 2/IRQ12
- J6 pad 68: /IRQ15 -> /Sheet 2/IRQ15
- J6 pad 69: /IRQ14 -> /Sheet 2/IRQ14
- J6 pad 70: /~{DACK0} -> /Sheet 2/~{DACK0}
- J6 pad 71: /DRQ0 -> /Sheet 2/DRQ0
- J6 pad 72: /~{DACK5} -> /Sheet 2/~{DACK5}
- J6 pad 73: /DRQ5 -> /Sheet 2/DRQ5
- J6 pad 74: /~{DACK6} -> /Sheet 2/~{DACK6}
- J6 pad 75: /DRQ6 -> /Sheet 2/DRQ6
- J6 pad 76: /~{DACK7} -> /Sheet 2/~{DACK7}
- J6 pad 77: /DRQ7 -> /Sheet 2/DRQ7
- J6 pad 79: /MASTER -> /Sheet 2/MASTER
- J6 pad 81: /SBHE -> /Sheet 2/SBHE
- J6 pad 82: /LA23 -> /Sheet 2/LA23
- J6 pad 83: /LA22 -> /Sheet 2/LA22
- J6 pad 84: /LA21 -> /Sheet 2/LA21
- J6 pad 85: /LA20 -> /Sheet 2/LA20
- J6 pad 86: /LA19 -> /Sheet 2/LA19
- J6 pad 87: /LA18 -> /Sheet 2/LA18
- J6 pad 88: /LA17 -> /Sheet 2/LA17
- J6 pad 89: /~{MEMR} -> /Sheet 2/~{MEMR}
- J6 pad 90: /~{MEMW} -> /Sheet 2/~{MEMW}
- J6 pad 91: /D8 -> /Sheet 2/D8
- J6 pad 92: /D9 -> /Sheet 2/D9
- J6 pad 93: /D10 -> /Sheet 2/D10
- J6 pad 94: /D11 -> /Sheet 2/D11
- J6 pad 95: /D12 -> /Sheet 2/D12
- J6 pad 96: /D13 -> /Sheet 2/D13
- J6 pad 97: /D14 -> /Sheet 2/D14
- J6 pad 98: /D15 -> /Sheet 2/D15
- J7 pad 11: /~{MEMWR} -> /Sheet 2/~{MEMWR}
- J7 pad 12: /~{MEMRD} -> /Sheet 2/~{MEMRD}
- J7 pad 13: /~{IOW} -> /Sheet 2/~{IOW}
- J7 pad 14: /~{IOR} -> /Sheet 2/~{IOR}
- J7 pad 15: /~{DACK3} -> /Sheet 2/~{DACK3}
- J7 pad 16: /DRQ3 -> /Sheet 2/DRQ3
- J7 pad 17: /~{DACK1} -> /Sheet 2/~{DACK1}
- J7 pad 18: /DRQ1 -> /Sheet 2/DRQ1
- J7 pad 19: /~{REFRESH} -> /Sheet 2/~{REFRESH}
- J7 pad 2: /RESET -> /Sheet 2/RESET
- J7 pad 20: /CLK -> /Sheet 2/CLK
- J7 pad 21: /IRQ7 -> /Sheet 2/IRQ7
- J7 pad 22: /IRQ6 -> /Sheet 2/IRQ6
- J7 pad 23: /IRQ5 -> /Sheet 2/IRQ5
- J7 pad 24: /IRQ4 -> /Sheet 2/IRQ4
- J7 pad 25: /IRQ3 -> /Sheet 2/IRQ3
- J7 pad 26: /~{DACK2} -> /Sheet 2/~{DACK2}
- J7 pad 27: /TC -> /Sheet 2/TC
- J7 pad 28: /ALE -> /Sheet 2/ALE
- J7 pad 30: /OSC -> /Sheet 2/OSC
- J7 pad 32: /IO -> /Sheet 2/IO
- J7 pad 33: /D7 -> /Sheet 2/D7
- J7 pad 34: /D6 -> /Sheet 2/D6
- J7 pad 35: /D5 -> /Sheet 2/D5
- J7 pad 36: /D4 -> /Sheet 2/D4
- J7 pad 37: /D3 -> /Sheet 2/D3
- J7 pad 38: /D2 -> /Sheet 2/D2
- J7 pad 39: /D1 -> /Sheet 2/D1
- J7 pad 4: /IRQ2 -> /Sheet 2/IRQ2
- J7 pad 40: /D0 -> /Sheet 2/D0
- J7 pad 41: /IORDY -> /Sheet 2/IORDY
- J7 pad 42: /AEN -> /Sheet 2/AEN
- J7 pad 43: /A19 -> /Sheet 2/A19
- J7 pad 44: /A18 -> /Sheet 2/A18
- J7 pad 45: /A17 -> /Sheet 2/A17
- J7 pad 46: /A16 -> /Sheet 2/A16
- J7 pad 47: /A15 -> /Sheet 2/A15
- J7 pad 48: /A14 -> /Sheet 2/A14
- J7 pad 49: /A13 -> /Sheet 2/A13
- J7 pad 50: /A12 -> /Sheet 2/A12
- J7 pad 51: /A11 -> /Sheet 2/A11
- J7 pad 52: /A10 -> /Sheet 2/A10
- J7 pad 53: /A9 -> /Sheet 2/A9
- J7 pad 54: /A8 -> /Sheet 2/A8
- J7 pad 55: /A7 -> /Sheet 2/A7
- J7 pad 56: /A6 -> /Sheet 2/A6
- J7 pad 57: /A5 -> /Sheet 2/A5
- J7 pad 58: /A4 -> /Sheet 2/A4
- J7 pad 59: /A3 -> /Sheet 2/A3
- J7 pad 6: /DRQ2 -> /Sheet 2/DRQ2
- J7 pad 60: /A2 -> /Sheet 2/A2
- J7 pad 61: /A1 -> /Sheet 2/A1
- J7 pad 62: /A0 -> /Sheet 2/A0
- J7 pad 63: /~{MEMCS16} -> /Sheet 2/~{MEMCS16}
- J7 pad 64: /~{IOCS16} -> /Sheet 2/~{IOCS16}
- J7 pad 65: /IRQ10 -> /Sheet 2/IRQ10
- J7 pad 66: /IRQ11 -> /Sheet 2/IRQ11
- J7 pad 67: /IRQ12 -> /Sheet 2/IRQ12
- J7 pad 68: /IRQ15 -> /Sheet 2/IRQ15
- J7 pad 69: /IRQ14 -> /Sheet 2/IRQ14
- J7 pad 70: /~{DACK0} -> /Sheet 2/~{DACK0}
- J7 pad 71: /DRQ0 -> /Sheet 2/DRQ0
- J7 pad 72: /~{DACK5} -> /Sheet 2/~{DACK5}
- J7 pad 73: /DRQ5 -> /Sheet 2/DRQ5
- J7 pad 74: /~{DACK6} -> /Sheet 2/~{DACK6}
- J7 pad 75: /DRQ6 -> /Sheet 2/DRQ6
- J7 pad 76: /~{DACK7} -> /Sheet 2/~{DACK7}
- J7 pad 77: /DRQ7 -> /Sheet 2/DRQ7
- J7 pad 79: /MASTER -> /Sheet 2/MASTER
- J7 pad 81: /SBHE -> /Sheet 2/SBHE
- J7 pad 82: /LA23 -> /Sheet 2/LA23
- J7 pad 83: /LA22 -> /Sheet 2/LA22
- J7 pad 84: /LA21 -> /Sheet 2/LA21
- J7 pad 85: /LA20 -> /Sheet 2/LA20
- J7 pad 86: /LA19 -> /Sheet 2/LA19
- J7 pad 87: /LA18 -> /Sheet 2/LA18
- J7 pad 88: /LA17 -> /Sheet 2/LA17
- J7 pad 89: /~{MEMR} -> /Sheet 2/~{MEMR}
- J7 pad 90: /~{MEMW} -> /Sheet 2/~{MEMW}
- J7 pad 91: /D8 -> /Sheet 2/D8
- J7 pad 92: /D9 -> /Sheet 2/D9
- J7 pad 93: /D10 -> /Sheet 2/D10
- J7 pad 94: /D11 -> /Sheet 2/D11
- J7 pad 95: /D12 -> /Sheet 2/D12
- J7 pad 96: /D13 -> /Sheet 2/D13
- J7 pad 97: /D14 -> /Sheet 2/D14
- J7 pad 98: /D15 -> /Sheet 2/D15
- J8 pad 11: /~{MEMWR} -> /Sheet 2/~{MEMWR}
- J8 pad 12: /~{MEMRD} -> /Sheet 2/~{MEMRD}
- J8 pad 13: /~{IOW} -> /Sheet 2/~{IOW}
- J8 pad 14: /~{IOR} -> /Sheet 2/~{IOR}
- J8 pad 15: /~{DACK3} -> /Sheet 2/~{DACK3}
- J8 pad 16: /DRQ3 -> /Sheet 2/DRQ3
- J8 pad 17: /~{DACK1} -> /Sheet 2/~{DACK1}
- J8 pad 18: /DRQ1 -> /Sheet 2/DRQ1
- J8 pad 19: /~{REFRESH} -> /Sheet 2/~{REFRESH}
- J8 pad 2: /RESET -> /Sheet 2/RESET
- J8 pad 20: /CLK -> /Sheet 2/CLK
- J8 pad 21: /IRQ7 -> /Sheet 2/IRQ7
- J8 pad 22: /IRQ6 -> /Sheet 2/IRQ6
- J8 pad 23: /IRQ5 -> /Sheet 2/IRQ5
- J8 pad 24: /IRQ4 -> /Sheet 2/IRQ4
- J8 pad 25: /IRQ3 -> /Sheet 2/IRQ3
- J8 pad 26: /~{DACK2} -> /Sheet 2/~{DACK2}
- J8 pad 27: /TC -> /Sheet 2/TC
- J8 pad 28: /ALE -> /Sheet 2/ALE
- J8 pad 30: /OSC -> /Sheet 2/OSC
- J8 pad 32: /IO -> /Sheet 2/IO
- J8 pad 33: /D7 -> /Sheet 2/D7
- J8 pad 34: /D6 -> /Sheet 2/D6
- J8 pad 35: /D5 -> /Sheet 2/D5
- J8 pad 36: /D4 -> /Sheet 2/D4
- J8 pad 37: /D3 -> /Sheet 2/D3
- J8 pad 38: /D2 -> /Sheet 2/D2
- J8 pad 39: /D1 -> /Sheet 2/D1
- J8 pad 4: /IRQ2 -> /Sheet 2/IRQ2
- J8 pad 40: /D0 -> /Sheet 2/D0
- J8 pad 41: /IORDY -> /Sheet 2/IORDY
- J8 pad 42: /AEN -> /Sheet 2/AEN
- J8 pad 43: /A19 -> /Sheet 2/A19
- J8 pad 44: /A18 -> /Sheet 2/A18
- J8 pad 45: /A17 -> /Sheet 2/A17
- J8 pad 46: /A16 -> /Sheet 2/A16
- J8 pad 47: /A15 -> /Sheet 2/A15
- J8 pad 48: /A14 -> /Sheet 2/A14
- J8 pad 49: /A13 -> /Sheet 2/A13
- J8 pad 50: /A12 -> /Sheet 2/A12
- J8 pad 51: /A11 -> /Sheet 2/A11
- J8 pad 52: /A10 -> /Sheet 2/A10
- J8 pad 53: /A9 -> /Sheet 2/A9
- J8 pad 54: /A8 -> /Sheet 2/A8
- J8 pad 55: /A7 -> /Sheet 2/A7
- J8 pad 56: /A6 -> /Sheet 2/A6
- J8 pad 57: /A5 -> /Sheet 2/A5
- J8 pad 58: /A4 -> /Sheet 2/A4
- J8 pad 59: /A3 -> /Sheet 2/A3
- J8 pad 6: /DRQ2 -> /Sheet 2/DRQ2
- J8 pad 60: /A2 -> /Sheet 2/A2
- J8 pad 61: /A1 -> /Sheet 2/A1
- J8 pad 62: /A0 -> /Sheet 2/A0
- J8 pad 63: /~{MEMCS16} -> /Sheet 2/~{MEMCS16}
- J8 pad 64: /~{IOCS16} -> /Sheet 2/~{IOCS16}
- J8 pad 65: /IRQ10 -> /Sheet 2/IRQ10
- J8 pad 66: /IRQ11 -> /Sheet 2/IRQ11
- J8 pad 67: /IRQ12 -> /Sheet 2/IRQ12
- J8 pad 68: /IRQ15 -> /Sheet 2/IRQ15
- J8 pad 69: /IRQ14 -> /Sheet 2/IRQ14
- J8 pad 70: /~{DACK0} -> /Sheet 2/~{DACK0}
- J8 pad 71: /DRQ0 -> /Sheet 2/DRQ0
- J8 pad 72: /~{DACK5} -> /Sheet 2/~{DACK5}
- J8 pad 73: /DRQ5 -> /Sheet 2/DRQ5
- J8 pad 74: /~{DACK6} -> /Sheet 2/~{DACK6}
- J8 pad 75: /DRQ6 -> /Sheet 2/DRQ6
- J8 pad 76: /~{DACK7} -> /Sheet 2/~{DACK7}
- J8 pad 77: /DRQ7 -> /Sheet 2/DRQ7
- J8 pad 79: /MASTER -> /Sheet 2/MASTER
- J8 pad 81: /SBHE -> /Sheet 2/SBHE
- J8 pad 82: /LA23 -> /Sheet 2/LA23
- J8 pad 83: /LA22 -> /Sheet 2/LA22
- J8 pad 84: /LA21 -> /Sheet 2/LA21
- J8 pad 85: /LA20 -> /Sheet 2/LA20
- J8 pad 86: /LA19 -> /Sheet 2/LA19
- J8 pad 87: /LA18 -> /Sheet 2/LA18
- J8 pad 88: /LA17 -> /Sheet 2/LA17
- J8 pad 89: /~{MEMR} -> /Sheet 2/~{MEMR}
- J8 pad 90: /~{MEMW} -> /Sheet 2/~{MEMW}
- J8 pad 91: /D8 -> /Sheet 2/D8
- J8 pad 92: /D9 -> /Sheet 2/D9
- J8 pad 93: /D10 -> /Sheet 2/D10
- J8 pad 94: /D11 -> /Sheet 2/D11
- J8 pad 95: /D12 -> /Sheet 2/D12
- J8 pad 96: /D13 -> /Sheet 2/D13
- J8 pad 97: /D14 -> /Sheet 2/D14
- J8 pad 98: /D15 -> /Sheet 2/D15

Commit message: Revert "Cleaned up schematic, broke layout"
This reverts commit 42e2edff88598cae901a53fb2aea1a81c84d528d.
Connections:
- J5 pad 11: /Sheet 2/~{MEMWR} -> /~{MEMWR}
- J5 pad 12: /Sheet 2/~{MEMRD} -> /~{MEMRD}
- J5 pad 13: /Sheet 2/~{IOW} -> /~{IOW}
- J5 pad 14: /Sheet 2/~{IOR} -> /~{IOR}
- J5 pad 15: /Sheet 2/~{DACK3} -> /~{DACK3}
- J5 pad 16: /Sheet 2/DRQ3 -> /DRQ3
- J5 pad 17: /Sheet 2/~{DACK1} -> /~{DACK1}
- J5 pad 18: /Sheet 2/DRQ1 -> /DRQ1
- J5 pad 19: /Sheet 2/~{REFRESH} -> /~{REFRESH}
- J5 pad 2: /Sheet 2/RESET -> /RESET
- J5 pad 20: /Sheet 2/CLK -> /CLK
- J5 pad 21: /Sheet 2/IRQ7 -> /IRQ7
- J5 pad 22: /Sheet 2/IRQ6 -> /IRQ6
- J5 pad 23: /Sheet 2/IRQ5 -> /IRQ5
- J5 pad 24: /Sheet 2/IRQ4 -> /IRQ4
- J5 pad 25: /Sheet 2/IRQ3 -> /IRQ3
- J5 pad 26: /Sheet 2/~{DACK2} -> /~{DACK2}
- J5 pad 27: /Sheet 2/TC -> /TC
- J5 pad 28: /Sheet 2/ALE -> /ALE
- J5 pad 30: /Sheet 2/OSC -> /OSC
- J5 pad 32: /Sheet 2/IO -> /IO
- J5 pad 33: /Sheet 2/D7 -> /D7
- J5 pad 34: /Sheet 2/D6 -> /D6
- J5 pad 35: /Sheet 2/D5 -> /D5
- J5 pad 36: /Sheet 2/D4 -> /D4
- J5 pad 37: /Sheet 2/D3 -> /D3
- J5 pad 38: /Sheet 2/D2 -> /D2
- J5 pad 39: /Sheet 2/D1 -> /D1
- J5 pad 4: /Sheet 2/IRQ2 -> /IRQ2
- J5 pad 40: /Sheet 2/D0 -> /D0
- J5 pad 41: /Sheet 2/IORDY -> /IORDY
- J5 pad 42: /Sheet 2/AEN -> /AEN
- J5 pad 43: /Sheet 2/A19 -> /A19
- J5 pad 44: /Sheet 2/A18 -> /A18
- J5 pad 45: /Sheet 2/A17 -> /A17
- J5 pad 46: /Sheet 2/A16 -> /A16
- J5 pad 47: /Sheet 2/A15 -> /A15
- J5 pad 48: /Sheet 2/A14 -> /A14
- J5 pad 49: /Sheet 2/A13 -> /A13
- J5 pad 50: /Sheet 2/A12 -> /A12
- J5 pad 51: /Sheet 2/A11 -> /A11
- J5 pad 52: /Sheet 2/A10 -> /A10
- J5 pad 53: /Sheet 2/A9 -> /A9
- J5 pad 54: /Sheet 2/A8 -> /A8
- J5 pad 55: /Sheet 2/A7 -> /A7
- J5 pad 56: /Sheet 2/A6 -> /A6
- J5 pad 57: /Sheet 2/A5 -> /A5
- J5 pad 58: /Sheet 2/A4 -> /A4
- J5 pad 59: /Sheet 2/A3 -> /A3
- J5 pad 6: /Sheet 2/DRQ2 -> /DRQ2
- J5 pad 60: /Sheet 2/A2 -> /A2
- J5 pad 61: /Sheet 2/A1 -> /A1
- J5 pad 62: /Sheet 2/A0 -> /A0
- J5 pad 63: /Sheet 2/~{MEMCS16} -> /~{MEMCS16}
- J5 pad 64: /Sheet 2/~{IOCS16} -> /~{IOCS16}
- J5 pad 65: /Sheet 2/IRQ10 -> /IRQ10
- J5 pad 66: /Sheet 2/IRQ11 -> /IRQ11
- J5 pad 67: /Sheet 2/IRQ12 -> /IRQ12
- J5 pad 68: /Sheet 2/IRQ15 -> /IRQ15
- J5 pad 69: /Sheet 2/IRQ14 -> /IRQ14
- J5 pad 70: /Sheet 2/~{DACK0} -> /~{DACK0}
- J5 pad 71: /Sheet 2/DRQ0 -> /DRQ0
- J5 pad 72: /Sheet 2/~{DACK5} -> /~{DACK5}
- J5 pad 73: /Sheet 2/DRQ5 -> /DRQ5
- J5 pad 74: /Sheet 2/~{DACK6} -> /~{DACK6}
- J5 pad 75: /Sheet 2/DRQ6 -> /DRQ6
- J5 pad 76: /Sheet 2/~{DACK7} -> /~{DACK7}
- J5 pad 77: /Sheet 2/DRQ7 -> /DRQ7
- J5 pad 79: /Sheet 2/MASTER -> /MASTER
- J5 pad 81: /Sheet 2/SBHE -> /SBHE
- J5 pad 82: /Sheet 2/LA23 -> /LA23
- J5 pad 83: /Sheet 2/LA22 -> /LA22
- J5 pad 84: /Sheet 2/LA21 -> /LA21
- J5 pad 85: /Sheet 2/LA20 -> /LA20
- J5 pad 86: /Sheet 2/LA19 -> /LA19
- J5 pad 87: /Sheet 2/LA18 -> /LA18
- J5 pad 88: /Sheet 2/LA17 -> /LA17
- J5 pad 89: /Sheet 2/~{MEMR} -> /~{MEMR}
- J5 pad 90: /Sheet 2/~{MEMW} -> /~{MEMW}
- J5 pad 91: /Sheet 2/D8 -> /D8
- J5 pad 92: /Sheet 2/D9 -> /D9
- J5 pad 93: /Sheet 2/D10 -> /D10
- J5 pad 94: /Sheet 2/D11 -> /D11
- J5 pad 95: /Sheet 2/D12 -> /D12
- J5 pad 96: /Sheet 2/D13 -> /D13
- J5 pad 97: /Sheet 2/D14 -> /D14
- J5 pad 98: /Sheet 2/D15 -> /D15
- J6 pad 11: /Sheet 2/~{MEMWR} -> /~{MEMWR}
- J6 pad 12: /Sheet 2/~{MEMRD} -> /~{MEMRD}
- J6 pad 13: /Sheet 2/~{IOW} -> /~{IOW}
- J6 pad 14: /Sheet 2/~{IOR} -> /~{IOR}
- J6 pad 15: /Sheet 2/~{DACK3} -> /~{DACK3}
- J6 pad 16: /Sheet 2/DRQ3 -> /DRQ3
- J6 pad 17: /Sheet 2/~{DACK1} -> /~{DACK1}
- J6 pad 18: /Sheet 2/DRQ1 -> /DRQ1
- J6 pad 19: /Sheet 2/~{REFRESH} -> /~{REFRESH}
- J6 pad 2: /Sheet 2/RESET -> /RESET
- J6 pad 20: /Sheet 2/CLK -> /CLK
- J6 pad 21: /Sheet 2/IRQ7 -> /IRQ7
- J6 pad 22: /Sheet 2/IRQ6 -> /IRQ6
- J6 pad 23: /Sheet 2/IRQ5 -> /IRQ5
- J6 pad 24: /Sheet 2/IRQ4 -> /IRQ4
- J6 pad 25: /Sheet 2/IRQ3 -> /IRQ3
- J6 pad 26: /Sheet 2/~{DACK2} -> /~{DACK2}
- J6 pad 27: /Sheet 2/TC -> /TC
- J6 pad 28: /Sheet 2/ALE -> /ALE
- J6 pad 30: /Sheet 2/OSC -> /OSC
- J6 pad 32: /Sheet 2/IO -> /IO
- J6 pad 33: /Sheet 2/D7 -> /D7
- J6 pad 34: /Sheet 2/D6 -> /D6
- J6 pad 35: /Sheet 2/D5 -> /D5
- J6 pad 36: /Sheet 2/D4 -> /D4
- J6 pad 37: /Sheet 2/D3 -> /D3
- J6 pad 38: /Sheet 2/D2 -> /D2
- J6 pad 39: /Sheet 2/D1 -> /D1
- J6 pad 4: /Sheet 2/IRQ2 -> /IRQ2
- J6 pad 40: /Sheet 2/D0 -> /D0
- J6 pad 41: /Sheet 2/IORDY -> /IORDY
- J6 pad 42: /Sheet 2/AEN -> /AEN
- J6 pad 43: /Sheet 2/A19 -> /A19
- J6 pad 44: /Sheet 2/A18 -> /A18
- J6 pad 45: /Sheet 2/A17 -> /A17
- J6 pad 46: /Sheet 2/A16 -> /A16
- J6 pad 47: /Sheet 2/A15 -> /A15
- J6 pad 48: /Sheet 2/A14 -> /A14
- J6 pad 49: /Sheet 2/A13 -> /A13
- J6 pad 50: /Sheet 2/A12 -> /A12
- J6 pad 51: /Sheet 2/A11 -> /A11
- J6 pad 52: /Sheet 2/A10 -> /A10
- J6 pad 53: /Sheet 2/A9 -> /A9
- J6 pad 54: /Sheet 2/A8 -> /A8
- J6 pad 55: /Sheet 2/A7 -> /A7
- J6 pad 56: /Sheet 2/A6 -> /A6
- J6 pad 57: /Sheet 2/A5 -> /A5
- J6 pad 58: /Sheet 2/A4 -> /A4
- J6 pad 59: /Sheet 2/A3 -> /A3
- J6 pad 6: /Sheet 2/DRQ2 -> /DRQ2
- J6 pad 60: /Sheet 2/A2 -> /A2
- J6 pad 61: /Sheet 2/A1 -> /A1
- J6 pad 62: /Sheet 2/A0 -> /A0
- J6 pad 63: /Sheet 2/~{MEMCS16} -> /~{MEMCS16}
- J6 pad 64: /Sheet 2/~{IOCS16} -> /~{IOCS16}
- J6 pad 65: /Sheet 2/IRQ10 -> /IRQ10
- J6 pad 66: /Sheet 2/IRQ11 -> /IRQ11
- J6 pad 67: /Sheet 2/IRQ12 -> /IRQ12
- J6 pad 68: /Sheet 2/IRQ15 -> /IRQ15
- J6 pad 69: /Sheet 2/IRQ14 -> /IRQ14
- J6 pad 70: /Sheet 2/~{DACK0} -> /~{DACK0}
- J6 pad 71: /Sheet 2/DRQ0 -> /DRQ0
- J6 pad 72: /Sheet 2/~{DACK5} -> /~{DACK5}
- J6 pad 73: /Sheet 2/DRQ5 -> /DRQ5
- J6 pad 74: /Sheet 2/~{DACK6} -> /~{DACK6}
- J6 pad 75: /Sheet 2/DRQ6 -> /DRQ6
- J6 pad 76: /Sheet 2/~{DACK7} -> /~{DACK7}
- J6 pad 77: /Sheet 2/DRQ7 -> /DRQ7
- J6 pad 79: /Sheet 2/MASTER -> /MASTER
- J6 pad 81: /Sheet 2/SBHE -> /SBHE
- J6 pad 82: /Sheet 2/LA23 -> /LA23
- J6 pad 83: /Sheet 2/LA22 -> /LA22
- J6 pad 84: /Sheet 2/LA21 -> /LA21
- J6 pad 85: /Sheet 2/LA20 -> /LA20
- J6 pad 86: /Sheet 2/LA19 -> /LA19
- J6 pad 87: /Sheet 2/LA18 -> /LA18
- J6 pad 88: /Sheet 2/LA17 -> /LA17
- J6 pad 89: /Sheet 2/~{MEMR} -> /~{MEMR}
- J6 pad 90: /Sheet 2/~{MEMW} -> /~{MEMW}
- J6 pad 91: /Sheet 2/D8 -> /D8
- J6 pad 92: /Sheet 2/D9 -> /D9
- J6 pad 93: /Sheet 2/D10 -> /D10
- J6 pad 94: /Sheet 2/D11 -> /D11
- J6 pad 95: /Sheet 2/D12 -> /D12
- J6 pad 96: /Sheet 2/D13 -> /D13
- J6 pad 97: /Sheet 2/D14 -> /D14
- J6 pad 98: /Sheet 2/D15 -> /D15
- J7 pad 11: /Sheet 2/~{MEMWR} -> /~{MEMWR}
- J7 pad 12: /Sheet 2/~{MEMRD} -> /~{MEMRD}
- J7 pad 13: /Sheet 2/~{IOW} -> /~{IOW}
- J7 pad 14: /Sheet 2/~{IOR} -> /~{IOR}
- J7 pad 15: /Sheet 2/~{DACK3} -> /~{DACK3}
- J7 pad 16: /Sheet 2/DRQ3 -> /DRQ3
- J7 pad 17: /Sheet 2/~{DACK1} -> /~{DACK1}
- J7 pad 18: /Sheet 2/DRQ1 -> /DRQ1
- J7 pad 19: /Sheet 2/~{REFRESH} -> /~{REFRESH}
- J7 pad 2: /Sheet 2/RESET -> /RESET
- J7 pad 20: /Sheet 2/CLK -> /CLK
- J7 pad 21: /Sheet 2/IRQ7 -> /IRQ7
- J7 pad 22: /Sheet 2/IRQ6 -> /IRQ6
- J7 pad 23: /Sheet 2/IRQ5 -> /IRQ5
- J7 pad 24: /Sheet 2/IRQ4 -> /IRQ4
- J7 pad 25: /Sheet 2/IRQ3 -> /IRQ3
- J7 pad 26: /Sheet 2/~{DACK2} -> /~{DACK2}
- J7 pad 27: /Sheet 2/TC -> /TC
- J7 pad 28: /Sheet 2/ALE -> /ALE
- J7 pad 30: /Sheet 2/OSC -> /OSC
- J7 pad 32: /Sheet 2/IO -> /IO
- J7 pad 33: /Sheet 2/D7 -> /D7
- J7 pad 34: /Sheet 2/D6 -> /D6
- J7 pad 35: /Sheet 2/D5 -> /D5
- J7 pad 36: /Sheet 2/D4 -> /D4
- J7 pad 37: /Sheet 2/D3 -> /D3
- J7 pad 38: /Sheet 2/D2 -> /D2
- J7 pad 39: /Sheet 2/D1 -> /D1
- J7 pad 4: /Sheet 2/IRQ2 -> /IRQ2
- J7 pad 40: /Sheet 2/D0 -> /D0
- J7 pad 41: /Sheet 2/IORDY -> /IORDY
- J7 pad 42: /Sheet 2/AEN -> /AEN
- J7 pad 43: /Sheet 2/A19 -> /A19
- J7 pad 44: /Sheet 2/A18 -> /A18
- J7 pad 45: /Sheet 2/A17 -> /A17
- J7 pad 46: /Sheet 2/A16 -> /A16
- J7 pad 47: /Sheet 2/A15 -> /A15
- J7 pad 48: /Sheet 2/A14 -> /A14
- J7 pad 49: /Sheet 2/A13 -> /A13
- J7 pad 50: /Sheet 2/A12 -> /A12
- J7 pad 51: /Sheet 2/A11 -> /A11
- J7 pad 52: /Sheet 2/A10 -> /A10
- J7 pad 53: /Sheet 2/A9 -> /A9
- J7 pad 54: /Sheet 2/A8 -> /A8
- J7 pad 55: /Sheet 2/A7 -> /A7
- J7 pad 56: /Sheet 2/A6 -> /A6
- J7 pad 57: /Sheet 2/A5 -> /A5
- J7 pad 58: /Sheet 2/A4 -> /A4
- J7 pad 59: /Sheet 2/A3 -> /A3
- J7 pad 6: /Sheet 2/DRQ2 -> /DRQ2
- J7 pad 60: /Sheet 2/A2 -> /A2
- J7 pad 61: /Sheet 2/A1 -> /A1
- J7 pad 62: /Sheet 2/A0 -> /A0
- J7 pad 63: /Sheet 2/~{MEMCS16} -> /~{MEMCS16}
- J7 pad 64: /Sheet 2/~{IOCS16} -> /~{IOCS16}
- J7 pad 65: /Sheet 2/IRQ10 -> /IRQ10
- J7 pad 66: /Sheet 2/IRQ11 -> /IRQ11
- J7 pad 67: /Sheet 2/IRQ12 -> /IRQ12
- J7 pad 68: /Sheet 2/IRQ15 -> /IRQ15
- J7 pad 69: /Sheet 2/IRQ14 -> /IRQ14
- J7 pad 70: /Sheet 2/~{DACK0} -> /~{DACK0}
- J7 pad 71: /Sheet 2/DRQ0 -> /DRQ0
- J7 pad 72: /Sheet 2/~{DACK5} -> /~{DACK5}
- J7 pad 73: /Sheet 2/DRQ5 -> /DRQ5
- J7 pad 74: /Sheet 2/~{DACK6} -> /~{DACK6}
- J7 pad 75: /Sheet 2/DRQ6 -> /DRQ6
- J7 pad 76: /Sheet 2/~{DACK7} -> /~{DACK7}
- J7 pad 77: /Sheet 2/DRQ7 -> /DRQ7
- J7 pad 79: /Sheet 2/MASTER -> /MASTER
- J7 pad 81: /Sheet 2/SBHE -> /SBHE
- J7 pad 82: /Sheet 2/LA23 -> /LA23
- J7 pad 83: /Sheet 2/LA22 -> /LA22
- J7 pad 84: /Sheet 2/LA21 -> /LA21
- J7 pad 85: /Sheet 2/LA20 -> /LA20
- J7 pad 86: /Sheet 2/LA19 -> /LA19
- J7 pad 87: /Sheet 2/LA18 -> /LA18
- J7 pad 88: /Sheet 2/LA17 -> /LA17
- J7 pad 89: /Sheet 2/~{MEMR} -> /~{MEMR}
- J7 pad 90: /Sheet 2/~{MEMW} -> /~{MEMW}
- J7 pad 91: /Sheet 2/D8 -> /D8
- J7 pad 92: /Sheet 2/D9 -> /D9
- J7 pad 93: /Sheet 2/D10 -> /D10
- J7 pad 94: /Sheet 2/D11 -> /D11
- J7 pad 95: /Sheet 2/D12 -> /D12
- J7 pad 96: /Sheet 2/D13 -> /D13
- J7 pad 97: /Sheet 2/D14 -> /D14
- J7 pad 98: /Sheet 2/D15 -> /D15
- J8 pad 11: /Sheet 2/~{MEMWR} -> /~{MEMWR}
- J8 pad 12: /Sheet 2/~{MEMRD} -> /~{MEMRD}
- J8 pad 13: /Sheet 2/~{IOW} -> /~{IOW}
- J8 pad 14: /Sheet 2/~{IOR} -> /~{IOR}
- J8 pad 15: /Sheet 2/~{DACK3} -> /~{DACK3}
- J8 pad 16: /Sheet 2/DRQ3 -> /DRQ3
- J8 pad 17: /Sheet 2/~{DACK1} -> /~{DACK1}
- J8 pad 18: /Sheet 2/DRQ1 -> /DRQ1
- J8 pad 19: /Sheet 2/~{REFRESH} -> /~{REFRESH}
- J8 pad 2: /Sheet 2/RESET -> /RESET
- J8 pad 20: /Sheet 2/CLK -> /CLK
- J8 pad 21: /Sheet 2/IRQ7 -> /IRQ7
- J8 pad 22: /Sheet 2/IRQ6 -> /IRQ6
- J8 pad 23: /Sheet 2/IRQ5 -> /IRQ5
- J8 pad 24: /Sheet 2/IRQ4 -> /IRQ4
- J8 pad 25: /Sheet 2/IRQ3 -> /IRQ3
- J8 pad 26: /Sheet 2/~{DACK2} -> /~{DACK2}
- J8 pad 27: /Sheet 2/TC -> /TC
- J8 pad 28: /Sheet 2/ALE -> /ALE
- J8 pad 30: /Sheet 2/OSC -> /OSC
- J8 pad 32: /Sheet 2/IO -> /IO
- J8 pad 33: /Sheet 2/D7 -> /D7
- J8 pad 34: /Sheet 2/D6 -> /D6
- J8 pad 35: /Sheet 2/D5 -> /D5
- J8 pad 36: /Sheet 2/D4 -> /D4
- J8 pad 37: /Sheet 2/D3 -> /D3
- J8 pad 38: /Sheet 2/D2 -> /D2
- J8 pad 39: /Sheet 2/D1 -> /D1
- J8 pad 4: /Sheet 2/IRQ2 -> /IRQ2
- J8 pad 40: /Sheet 2/D0 -> /D0
- J8 pad 41: /Sheet 2/IORDY -> /IORDY
- J8 pad 42: /Sheet 2/AEN -> /AEN
- J8 pad 43: /Sheet 2/A19 -> /A19
- J8 pad 44: /Sheet 2/A18 -> /A18
- J8 pad 45: /Sheet 2/A17 -> /A17
- J8 pad 46: /Sheet 2/A16 -> /A16
- J8 pad 47: /Sheet 2/A15 -> /A15
- J8 pad 48: /Sheet 2/A14 -> /A14
- J8 pad 49: /Sheet 2/A13 -> /A13
- J8 pad 50: /Sheet 2/A12 -> /A12
- J8 pad 51: /Sheet 2/A11 -> /A11
- J8 pad 52: /Sheet 2/A10 -> /A10
- J8 pad 53: /Sheet 2/A9 -> /A9
- J8 pad 54: /Sheet 2/A8 -> /A8
- J8 pad 55: /Sheet 2/A7 -> /A7
- J8 pad 56: /Sheet 2/A6 -> /A6
- J8 pad 57: /Sheet 2/A5 -> /A5
- J8 pad 58: /Sheet 2/A4 -> /A4
- J8 pad 59: /Sheet 2/A3 -> /A3
- J8 pad 6: /Sheet 2/DRQ2 -> /DRQ2
- J8 pad 60: /Sheet 2/A2 -> /A2
- J8 pad 61: /Sheet 2/A1 -> /A1
- J8 pad 62: /Sheet 2/A0 -> /A0
- J8 pad 63: /Sheet 2/~{MEMCS16} -> /~{MEMCS16}
- J8 pad 64: /Sheet 2/~{IOCS16} -> /~{IOCS16}
- J8 pad 65: /Sheet 2/IRQ10 -> /IRQ10
- J8 pad 66: /Sheet 2/IRQ11 -> /IRQ11
- J8 pad 67: /Sheet 2/IRQ12 -> /IRQ12
- J8 pad 68: /Sheet 2/IRQ15 -> /IRQ15
- J8 pad 69: /Sheet 2/IRQ14 -> /IRQ14
- J8 pad 70: /Sheet 2/~{DACK0} -> /~{DACK0}
- J8 pad 71: /Sheet 2/DRQ0 -> /DRQ0
- J8 pad 72: /Sheet 2/~{DACK5} -> /~{DACK5}
- J8 pad 73: /Sheet 2/DRQ5 -> /DRQ5
- J8 pad 74: /Sheet 2/~{DACK6} -> /~{DACK6}
- J8 pad 75: /Sheet 2/DRQ6 -> /DRQ6
- J8 pad 76: /Sheet 2/~{DACK7} -> /~{DACK7}
- J8 pad 77: /Sheet 2/DRQ7 -> /DRQ7
- J8 pad 79: /Sheet 2/MASTER -> /MASTER
- J8 pad 81: /Sheet 2/SBHE -> /SBHE
- J8 pad 82: /Sheet 2/LA23 -> /LA23
- J8 pad 83: /Sheet 2/LA22 -> /LA22
- J8 pad 84: /Sheet 2/LA21 -> /LA21
- J8 pad 85: /Sheet 2/LA20 -> /LA20
- J8 pad 86: /Sheet 2/LA19 -> /LA19
- J8 pad 87: /Sheet 2/LA18 -> /LA18
- J8 pad 88: /Sheet 2/LA17 -> /LA17
- J8 pad 89: /Sheet 2/~{MEMR} -> /~{MEMR}
- J8 pad 90: /Sheet 2/~{MEMW} -> /~{MEMW}
- J8 pad 91: /Sheet 2/D8 -> /D8
- J8 pad 92: /Sheet 2/D9 -> /D9
- J8 pad 93: /Sheet 2/D10 -> /D10
- J8 pad 94: /Sheet 2/D11 -> /D11
- J8 pad 95: /Sheet 2/D12 -> /D12
- J8 pad 96: /Sheet 2/D13 -> /D13
- J8 pad 97: /Sheet 2/D14 -> /D14
- J8 pad 98: /Sheet 2/D15 -> /D15
