File: 286TowerOfSomething/isa-card/16bit-no-port/16bit-no-port.kicad_sch (KiCad schematic)
At the start: 2 parts, among them J1 Bus_ISA_16bit

Commit message: Adding Keystone 9200 bracket, and fixing refdes on no-port ISA card
Parts:
- renumbered U1 to BRACKET1
Changed lines of the file:
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@@
 		(dnp no)
 		(fields_autoplaced yes)
-		(property "Reference" "U1"
+		(property "Reference" "BRACKET1"
 			(at 163.83 186.69 0)
 			(effects
@@
 			(project ""
 				(path "/c4dfd9b2-d574-417c-9499-e52b1d483baa"
-					(reference "U1")
+					(reference "BRACKET1")
 					(unit 1)
 				)
