File: 286TowerOfSomething/isa-card/16bit-one-db9/16bit-one-db9.kicad_pcb (KiCad board)
At the start: 2 copper layers, 242.4 x 106.7 mm, 3 parts, among them J1 Bus_ISA_16bit, J2 DE9_Receptacle_MountingHoles

Commit message: Fixing refdes on one db9 card template
Parts:
- renumbered U1 to BRACKET1
Changed lines of the file:
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@@
 		)
 		(sheetname "Root")
-		(sheetfile "16bit-two-db9.kicad_sch")
+		(sheetfile "16bit-one-db9.kicad_sch")
 		(attr exclude_from_pos_files)
 		(fp_line
@@
 		(descr "Mounting Hole 3.2mm, M3")
 		(tags "mounting hole 3.2mm m3")
-		(property "Reference" "U1"
+		(property "Reference" "BRACKET1"
 			(at 20.35275 -16.082 0)
 			(layer "F.SilkS")
@@
 		)
 		(sheetname "Root")
-		(sheetfile "16bit-two-db9.kicad_sch")
+		(sheetfile "16bit-one-db9.kicad_sch")
 		(attr exclude_from_pos_files)
 		(fp_line
@@
 		(property ki_fp_filters "DSUB*Female*")
 		(sheetname "Root")
-		(sheetfile "16bit-two-db9.kicad_sch")
+		(sheetfile "16bit-one-db9.kicad_sch")
 		(attr through_hole)
 		(fp_line
