File: 286TowerOfSomething/isa-card/16bit-one-db9/16bit-one-db9.kicad_sch (KiCad schematic)
At the start: 3 parts, among them J1 Bus_ISA_16bit, J2 DE9_Receptacle_MountingHoles

Commit message: Fixing refdes on one db9 card template
Parts:
- renumbered U1 to BRACKET1
Changed lines of the file:
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@@
 		(dnp no)
 		(fields_autoplaced yes)
-		(property "Reference" "U1"
+		(property "Reference" "BRACKET1"
 			(at 163.83 186.69 0)
 			(effects
@@
 			(project ""
 				(path "/c4dfd9b2-d574-417c-9499-e52b1d483baa"
-					(reference "U1")
+					(reference "BRACKET1")
 					(unit 1)
 				)
