File: 286TowerOfSomething/isa-card/8bit-no-port/8bit-no-port.kicad_sch (KiCad schematic)
At the start: 2 parts, among them J1 Bus_ISA_8bit

Commit message: Updating 8-bit template to fix refdes
Parts:
- renumbered U1 to BRACKET1
Changed lines of the file:
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@@
 		(dnp no)
 		(fields_autoplaced yes)
-		(property "Reference" "U1"
+		(property "Reference" "BRACKET1"
 			(at 163.83 186.69 0)
 			(effects
@@
 			(project ""
 				(path "/c4dfd9b2-d574-417c-9499-e52b1d483baa"
-					(reference "U1")
+					(reference "BRACKET1")
 					(unit 1)
 				)
