File: dmp-go-away/npu.kicad_sch (KiCad schematic)
At the start: 3 parts, among them U1 M6117C

Commit message: Adding layout of dmp-go-away in progress
Changed lines of the file:
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@@
 (kicad_sch
-	(version 20231120)
+	(version 20250114)
 	(generator "eeschema")
-	(generator_version "8.0")
+	(generator_version "9.0")
 	(paper "USLetter")
 	(wire
@@
 		(shape bidirectional)
 		(at 140.97 102.87 0)
-		(fields_autoplaced yes)
 		(effects
 			(font
@@
 		(shape bidirectional)
 		(at 140.97 97.79 0)
-		(fields_autoplaced yes)
 		(effects
 			(font
