File: dmp-go-away/oscillator.kicad_sch (KiCad schematic)
At the start: 14 parts, among them Q1 MMBT3904, U1 M6117C, X1 80.000 MHz, X2 14.318 MHz

Commit message: Adding layout of dmp-go-away in progress
Changed lines of the file:
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@@
 (kicad_sch
-	(version 20231120)
+	(version 20250114)
 	(generator "eeschema")
-	(generator_version "8.0")
+	(generator_version "9.0")
 	(paper "USLetter")
 	(junction
@@
 		(shape bidirectional)
 		(at 101.6 97.79 0)
-		(fields_autoplaced yes)
 		(effects
 			(font
@@
 		(shape input)
 		(at 50.8 87.63 180)
-		(fields_autoplaced yes)
 		(effects
 			(font
@@
 		(shape bidirectional)
 		(at 50.8 90.17 180)
-		(fields_autoplaced yes)
 		(effects
 			(font
@@
 		(shape bidirectional)
 		(at 135.89 127 0)
-		(fields_autoplaced yes)
 		(effects
 			(font
@@
 		(shape bidirectional)
 		(at 135.89 81.28 0)
-		(fields_autoplaced yes)
 		(effects
 			(font
@@
 		(shape bidirectional)
 		(at 101.6 92.71 0)
-		(fields_autoplaced yes)
 		(effects
 			(font
