File: dmp-go-away/ram.kicad_sch (KiCad schematic)
At the start: 34 parts, among them U1 M6117C, U2 M5M416160CJ, U3 M5M416160CJ, U4 M5M416160CJ, U5 M5M416160CJ

Commit message: Adding layout of dmp-go-away in progress
Connections:
- net ~{LCAS0} is gone; now on net ~{CAS0L}: U2.31 (~{LCAS})
- net ~{LCAS1} is gone; now on net ~{CAS1L}: U3.31 (~{LCAS})
- net ~{LCAS2} is gone; now on net ~{CAS2L}: U4.31 (~{LCAS})
- net ~{LCAS3} is gone; now on net ~{CAS3L}: U5.31 (~{LCAS})
- net ~{UCAS0} is gone; now on net ~{CAS0H}: U2.30 (~{UCAS})
- net ~{UCAS1} is gone; now on net ~{CAS1H}: U3.30 (~{UCAS})
- net ~{UCAS2} is gone; now on net ~{CAS2H}: U4.30 (~{UCAS})
- net ~{UCAS3} is gone; now on net ~{CAS3H}: U5.30 (~{UCAS})
