File: dmp-go-away/dmp-go-away.kicad_pcb (KiCad board)
At the start: 2 copper layers, 242.4 x 106.7 mm, 92 parts, among them J1 Bus_ISA_16bit, J2 Conn_02x20_Odd_Even, J3 Keyboard, J4 Mouse, Q1 MMBT3904, U1 M6117C, U2 M5M416160CJ, U3 M5M416160CJ, U4 M5M416160CJ, U5 M5M416160CJ, U6 SST39SF010, U7 74LS245, U8 74LS245, U9 DS12885, X1 80.000 MHz, X2 14.318 MHz, Y1 32.768 kHz, Y2 32.768 kHz

Commit message: Adding layout of dmp-go-away in progress
Parts:
- C1, C2, C3, C33, C4, R1, R10, R11, R12, R13, R14, R15, R16, R17, R18, R19, R2, R20, R21, R22, R23, R24, R25, R3, R4, R5, R6, R7, R8, R9, U1, U2, U3, U4, U5, X2: moved to B.Cu
- moved R2 426.2 mm to (195.6, 62.2), turned to -90 degrees
- moved R3 424.2 mm to (194.1, 62.2), turned to -90 degrees
- moved R4 422.1 mm to (192.5, 62.2), turned to -90 degrees
- moved R5 420.6 mm to (191.0, 62.2), turned to -90 degrees
- moved R6 418.5 mm to (189.5, 62.2), turned to -90 degrees
- moved R7 416.4 mm to (188.0, 62.2), turned to -90 degrees
- moved R8 414.3 mm to (186.4, 62.2), turned to -90 degrees
- moved R9 412.2 mm to (184.9, 62.2), turned to -90 degrees
- moved R10 410.1 mm to (183.4, 62.2), turned to -90 degrees
- moved R11 408.0 mm to (181.9, 62.2), turned to -90 degrees
- moved R12 406.0 mm to (180.3, 62.2), turned to -90 degrees
- moved R13 404.6 mm to (178.8, 62.2), turned to -90 degrees
- moved R18 400.0 mm to (177.3, 62.2), turned to -90 degrees
- moved R19 397.9 mm to (175.8, 62.2), turned to -90 degrees
- moved U2 397.7 mm to (190.5, 45.7), turned to -90 degrees
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Connections:
- U2 pad 30: /RAM/~{UCAS0} -> /RAM/~{CAS0H}
- U2 pad 31: /RAM/~{LCAS0} -> /RAM/~{CAS0L}
- U3 pad 30: /RAM/~{UCAS1} -> /RAM/~{CAS1H}
- U3 pad 31: /RAM/~{LCAS1} -> /RAM/~{CAS1L}
- U4 pad 30: /RAM/~{UCAS2} -> /RAM/~{CAS2H}
- U4 pad 31: /RAM/~{LCAS2} -> /RAM/~{CAS2L}
- U5 pad 30: /RAM/~{UCAS3} -> /RAM/~{CAS3H}
- U5 pad 31: /RAM/~{LCAS3} -> /RAM/~{CAS3L}
Routing:
- net /~{IOCHK}: track 0.00 -> 105.3 mm, vias 0 -> 3
- net /RAM/D15: track 0.00 -> 102.1 mm, vias 0 -> 2
- net /RAM/D14: track 0.00 -> 100.7 mm, vias 0 -> 2
- net /RAM/D13: track 0.00 -> 98.8 mm, vias 0 -> 2
- net /RAM/D12: track 0.00 -> 97.0 mm, vias 0 -> 2
- net /RAM/D1: track 0.00 -> 96.7 mm, vias 0 -> 2
- net /RAM/D0: track 0.00 -> 96.4 mm, vias 0 -> 2
- net /RAM/D2: track 0.00 -> 95.8 mm, vias 0 -> 2
- net /RAM/D3: track 0.00 -> 95.0 mm, vias 0 -> 2
- net /RAM/D11: track 0.00 -> 93.9 mm, vias 0 -> 2
- net /SD7: track 0.00 -> 93.3 mm, vias 0 -> 1
- net /RAM/D4: track 0.00 -> 93.0 mm, vias 0 -> 2
- net /RAM/D10: track 0.00 -> 92.3 mm, vias 0 -> 2
- net /RAM/D5: track 0.00 -> 92.1 mm, vias 0 -> 2
- net /RAM/D6: track 0.00 -> 91.3 mm, vias 0 -> 2
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
Commit message: Adding IDE fixes and some layout work
Parts:
- C1, C2, C3, C33, C4, R1, R10, R11, R12, R13, R14, R15, R16, R17, R18, R19, R2, R20, R21, R22, R23, R24, R25, R3, R4, R5, R6, R7, R8, R9, U1, U2, U3, U4, U5, X2: moved to F.Cu
- C10, C11, C12, C13, C14, C15, C16, C17, C18, C19, C20, C21, C22, C30, C8, C9, R29: moved to B.Cu
- U7, U8: footprint Package_SO:SSOP-20_5.3x7.2mm_P0.65mm -> Package_SO:SOIC-20W_7.5x12.8mm_P1.27mm
- moved U6 330.6 mm to (195.6, 102.9), turned to 180 degrees
- moved Y2 307.1 mm to (226.3, 90.2), turned to 90 degrees
- moved U9 299.3 mm to (221.2, 92.7), turned to 180 degrees
- moved C35 258.3 mm to (202.2, 85.1), turned to 180 degrees
- moved C34 253.3 mm to (202.2, 77.5), turned to 180 degrees
- moved R31 251.8 mm to (202.2, 74.9), turned to 0 degrees
- moved C24 235.6 mm to (157.2, 54.1), turned to 180 degrees
- moved C23 234.7 mm to (144.8, 56.1)
- moved U8 233.2 mm to (165.1, 48.3), turned to 180 degrees
- moved J2 221.7 mm to (139.7, 35.6), turned to 90 degrees
- moved U7 219.7 mm to (144.8, 48.3)
- moved JP3 217.5 mm to (137.4, 53.5), turned to 90 degrees
- moved JP4 203.8 mm to (137.4, 43.2), turned to 90 degrees
- moved JP1 195.4 mm to (188.0, 41.1), turned to 90 degrees
- moved JP2 180.9 mm to (184.2, 41.1), turned to 90 degrees
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Routing:
- net /~{IOCHK}: track 105.3 -> 0.00 mm, vias 3 -> 0
- net /RESETDRV: track 91.0 -> 0.00 mm, vias 2 -> 0
- net Net-(U1E-MSDATA/IRQ12): track 88.1 -> 0.00 mm
- net /IRQ9: track 87.6 -> 0.00 mm, vias 2 -> 0
- net Net-(U1E-KBDATA): track 87.4 -> 0.00 mm
- net /AEN: track 84.4 -> 0.00 mm, vias 1 -> 0
- net Net-(U1E-KBCLK): track 81.7 -> 0.00 mm
- net /SA0: track 28.3 -> 104.8 mm, vias 1 -> 2
- net /SA1: track 30.0 -> 100.8 mm, vias 1 -> 2
- net /IRQ10: track 70.5 -> 0.00 mm, vias 2 -> 0
- net /~{MASTER}: track 69.0 -> 0.00 mm, vias 2 -> 0
- net /~{SMEMW}: track 69.0 -> 0.00 mm, vias 2 -> 0
- net /IOCHRDY: track 68.6 -> 0.00 mm, vias 1 -> 0
- net /~{SMEMR}: track 65.8 -> 0.00 mm, vias 2 -> 0
- net /SA2: track 31.9 -> 96.8 mm, vias 1 -> 2
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