File: ethermaker/ethermaker.kicad_pcb (KiCad board)
At the start: 2 copper layers, 159.9 x 75.6 mm, 30 parts, among them J1 Bus_ISA_16bit, J2 RJ45_Hanrun_HR911105A_Horizon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, U1 CS8900A, U2 GAL16V8, U3 93C46A, U4 SST39SF010, U5 74LS245, Y1 20.0 MHz

Commit message: Adding ethermaker board updates
Routing:
- net /A12: track 124.6 -> 108.1 mm
Other:
- board size 159.9 x 75.6 mm -> 158.7 x 75.6 mm
- board text added: "Ethermaker 2025-04-11 by rglenn"
