File: flop-tonight/flop-tonight.kicad_sch (KiCad schematic)
At the start: 23 parts, among them J1 Bus_ISA_8bit, J2 Conn_02x17_Odd_Even, U1 PC8477BV, U2 74ALS138, U3 74ALS138, Y1 24 MHz

Commit message: Adding flop-tonight updates
Parts:
- added BRACKET1: ~, pc-parts:PC_BRACKET_ISA_KEYSTONE_9202_Rev1, symbol pc-parts:9202
Connections:
- net A5: now also U2.6 (E3); no longer U3.3 (A2)
- net A9: now also U3.3 (A2); no longer U2.6 (E3)
Changed lines of the file:
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@@
 (kicad_sch
-	(version 20231120)
+	(version 20250114)
 	(generator "eeschema")
-	(generator_version "8.0")
+	(generator_version "9.0")
 	(paper "USLetter")
 	(title_block
@@
 	(label "~{IOR}"
 		(at 20.32 58.42 0)
-		(fields_autoplaced yes)
 		(effects
 			(font
@@
 	(label "D0"
 		(at 114.3 45.72 0)
-		(fields_autoplaced yes)
 		(effects
 			(font
@@
 	(label "D0"
 		(at 81.28 45.72 180)
-		(fields_autoplaced yes)
 		(effects
 			(font
@@
 	(label "A7"
 		(at 31.75 161.29 0)
-		(fields_autoplaced yes)
 		(effects
 			(font
@@
 	(label "~{IOW}"
 		(at 114.3 81.28 0)
-		(fields_autoplaced yes)
 		(effects
 			(font
@@
 	(label "DRQ2"
 		(at 114.3 91.44 0)
-		(fields_autoplaced yes)
 		(effects
 			(font
@@
 	(label "A4"
 		(at 31.75 125.73 0)
-		(fields_autoplaced yes)
 		(effects
 			(font
@@
 	(label "RESET"
 		(at 20.32 27.94 0)
-		(fields_autoplaced yes)
 		(effects
 			(font
@@
 	(label "A4"
 		(at 81.28 91.44 180)
-		(fields_autoplaced yes)
 		(effects
 			(font
@@
 	(label "A7"
 		(at 81.28 83.82 180)
-		(fields_autoplaced yes)
 		(effects
 			(font
@@
 	(label "A6"
 		(at 31.75 163.83 0)
-		(fields_autoplaced yes)
 		(effects
 			(font
@@
 	(label "A8"
 		(at 81.28 81.28 180)
-		(fields_autoplaced yes)
 		(effects
 			(font
@@
 	(label "D2"
 		(at 81.28 40.64 180)
-		(fields_autoplaced yes)
 		(effects
 			(font
@@
 		)
 	)
-	(label "A9"
+	(label "A5"
 		(at 31.75 135.89 0)
-		(fields_autoplaced yes)
 		(effects
 			(font
@@
 	(label "A0"
 		(at 114.3 68.58 0)
-		(fields_autoplaced yes)
 		(effects
 			(font
@@
 	(label "A1"
 		(at 114.3 71.12 0)
-		(fields_autoplaced yes)
 		(effects
 			(font
@@
 	(label "~{FLOPPY_CS}"
 		(at 114.3 83.82 0)
-		(fields_autoplaced yes)
 		(effects
 			(font
@@
 	(label "A3"
 		(at 81.28 93.98 180)
-		(fields_autoplaced yes)
 		(effects
 			(font
@@
 	(label "D4"
 		(at 81.28 35.56 180)
-		(fields_autoplaced yes)
 		(effects
 			(font
@@
 	(label "~{IOW}"
 		(at 20.32 55.88 0)
-		(fields_autoplaced yes)
 		(effects
 			(font
@@
 	(label "D6"
 		(at 81.28 30.48 180)
-		(fields_autoplaced yes)
 		(effects
 			(font
@@
 	(label "A1"
 		(at 81.28 99.06 180)
-		(fields_autoplaced yes)
 		(effects
 			(font
@@
 	(label "D2"
 		(at 114.3 50.8 0)
-		(fields_autoplaced yes)
 		(effects
 			(font
@@
 	(label "AEN"
 		(at 31.75 140.97 0)
-		(fields_autoplaced yes)
 		(effects
 			(font
@@
 	(label "~{FLOPPY_CS}"
 		(at 73.66 130.81 180)
-		(fields_autoplaced yes)
 		(effects
 			(font
@@
 	(label "D3"
 		(at 81.28 38.1 180)
-		(fields_autoplaced yes)
 		(effects
 			(font
@@
 	(label "D5"
 		(at 114.3 58.42 0)
-		(fields_autoplaced yes)
 		(effects
 			(font
@@
 	(label "RESET"
 		(at 114.3 33.02 0)
-		(fields_autoplaced yes)
 		(effects
 			(font
@@
 	(label "~{DACK2}"
 		(at 114.3 88.9 0)
-		(fields_autoplaced yes)
 		(effects
 			(font
@@
 	(label "AEN"
 		(at 81.28 50.8 180)
-		(fields_autoplaced yes)
 		(effects
 			(font
@@
 	(label "A3"
 		(at 31.75 128.27 0)
-		(fields_autoplaced yes)
 		(effects
 			(font
@@
 	(label "DRQ2"
 		(at 20.32 38.1 0)
-		(fields_autoplaced yes)
 		(effects
 			(font
@@
 	(label "D5"
 		(at 81.28 33.02 180)
-		(fields_autoplaced yes)
 		(effects
 			(font
@@
 	(label "D1"
 		(at 81.28 43.18 180)
-		(fields_autoplaced yes)
 		(effects
 			(font
@@
 	(label "~{DACK2}"
 		(at 20.32 88.9 0)
-		(fields_autoplaced yes)
 		(effects
 			(font
@@
 	(label "IRQ6"
 		(at 114.3 99.06 0)
-		(fields_autoplaced yes)
 		(effects
 			(font
@@
 	(label "IRQ6"
 		(at 20.32 78.74 0)
-		(fields_autoplaced yes)
 		(effects
 			(font
@@
 	(label "D7"
 		(at 114.3 63.5 0)
-		(fields_autoplaced yes)
 		(effects
 			(font
@@
 	(label "A2"
 		(at 81.28 96.52 180)
-		(fields_autoplaced yes)
 		(effects
 			(font
@@
 	(label "D7"
 		(at 81.28 27.94 180)
-		(fields_autoplaced yes)
 		(effects
 			(font
@@
 	(label "D3"
 		(at 114.3 53.34 0)
-		(fields_autoplaced yes)
 		(effects
 			(font
@@
 	(label "D4"
 		(at 114.3 55.88 0)
-		(fields_autoplaced yes)
 		(effects
 			(font
@@
 	(label "~{IOR}"
 		(at 114.3 78.74 0)
-		(fields_autoplaced yes)
 		(effects
 			(font
@@
 	(label "A2"
 		(at 114.3 73.66 0)
-		(fields_autoplaced yes)
 		(effects
 			(font
@@
 	(label "D6"
 		(at 114.3 60.96 0)
-		(fields_autoplaced yes)
 		(effects
 			(font
@@
 	(label "A6"
 		(at 81.28 86.36 180)
-		(fields_autoplaced yes)
 		(effects
 			(font
@@
 	(label "A9"
 		(at 81.28 78.74 180)
-		(fields_autoplaced yes)
 		(effects
 			(font
@@
 	(label "D1"
 		(at 114.3 48.26 0)
-		(fields_autoplaced yes)
 		(effects
 			(font
@@
 	(label "A0"
 		(at 81.28 101.6 180)
-		(fields_autoplaced yes)
 		(effects
 			(font
@@
 	(label "A8"
 		(at 31.75 123.19 0)
-		(fields_autoplaced yes)
 		(effects
 			(font
@@
 	(label "TC"
 		(at 20.32 91.44 0)
-		(fields_autoplaced yes)
 		(effects
 			(font
@@
 	(label "A5"
 		(at 81.28 88.9 180)
-		(fields_autoplaced yes)
 		(effects
 			(font
@@
 		)
 	)
-	(label "A5"
+	(label "A9"
 		(at 31.75 166.37 0)
-		(fields_autoplaced yes)
 		(effects
 			(font
@@
 	(label "TC"
 		(at 114.3 93.98 0)
-		(fields_autoplaced yes)
 		(effects
 			(font
@@
 	)
 	(symbol
+		(lib_id "pc-parts:9202")
+		(at 245.11 134.62 0)
+		(unit 1)
+		(exclude_from_sim no)
+		(in_bom yes)
+		(on_board yes)
+		(dnp no)
+		(fields_autoplaced yes)
+		(property "Reference" "BRACKET1"
+			(at 245.11 134.62 0)
+			(effects
+				(font
+					(size 1.27 1.27)
+				)
+				(hide yes)
+			)
+		)
+		(property "Value" "~"
+			(at 250.19 134.62 0)
+			(effects
+				(font
+					(size 1.27 1.27)
+				)
+				(justify left)
+			)
+		)
+		(property "Footprint" "pc-parts:PC_BRACKET_ISA_KEYSTONE_9202_Rev1"
+			(at 245.11 134.62 0)
+			(effects
+				(font
+					(size 1.27 1.27)
+				)
+				(hide yes)
+			)
+		)
+		(property "Datasheet" ""
+			(at 245.11 134.62 0)
+			(effects
+				(font
+					(size 1.27 1.27)
+				)
+				(hide yes)
+			)
+		)
+		(property "Description" ""
+			(at 245.11 134.62 0)
+			(effects
+				(font
+					(size 1.27 1.27)
+				)
+				(hide yes)
+			)
+		)
+		(instances
+			(project "flop-tonight"
+				(path "/083e3fae-b4c5-4662-b26b-2f9fc6b9c9fc"
+					(reference "BRACKET1")
+					(unit 1)
+				)
+			)
+		)
+	)
+	(symbol
 		(lib_id "Connector:Bus_ISA_8bit")
 		(at 50.8 63.5 0)
@@
 		)
 	)
+	(embedded_fonts no)
 )
