File: go-lpt-it-out/go-lpt-it-out.kicad_pcb (KiCad board)
At the start: 2 copper layers, 108.3 x 89.9 mm, 46 parts, among them J1 Bus_ISA_8bit, J2 DE9, J3 Parallel, J4 Conn_02x05_Odd_Even, Q1 MMBT3904, SW1 SW_DIP_x06, SW2 SW_DIP_x07, U1 TL16C552A, U2 GD75232N, U3 GD75232N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

Commit message: Adding updates to go-lpt-it-out
Parts:
- J2: footprint Connector_Dsub:DSUB-9_Male_Horizontal_P2.77x2.84mm_EdgePinOffset4.94mm_Housed_MountingHolesOffset4.94mm -> Connector_Dsub:DSUB-9_Pins_Horizontal_P2.77x2.84mm_EdgePinOffset7.70mm_Housed_MountingHolesOffset9.12mm
- J3: footprint Connector_Dsub:DSUB-25_Female_Horizontal_P2.77x2.84mm_EdgePinOffset4.94mm_Housed_MountingHolesOffset4.94mm -> Connector_Dsub:DSUB-25_Socket_Horizontal_P2.77x2.84mm_EdgePinOffset7.70mm_Housed_MountingHolesOffset9.12mm
- moved J2 2.80 mm to (136.5, 103.4)
- moved J3 2.80 mm to (136.5, 125.4)
Routing:
- net /PARPORT_PE: track 80.9 -> 77.3 mm
- net /PARPORT_PD2: track 30.1 -> 26.8 mm
- net /PARPORT_PD1: track 27.6 -> 24.3 mm
- net /PARPORT_PD3: track 26.3 -> 23.1 mm
- net /PARPORT_PD4: track 28.7 -> 25.5 mm
- net /PARPORT_BUSY: track 76.7 -> 73.6 mm
- net /PARPORT_PD0: track 31.1 -> 28.0 mm
- net /~{PARPORT_ERR}: track 60.3 -> 57.2 mm
- net /~{PARPORT_ACK}: track 79.7 -> 76.7 mm
- net /PARPORT_SLCT: track 81.5 -> 78.7 mm
- net /~{PARPORT_AFD}: track 34.6 -> 31.8 mm
- net /PARPORT_PD5: track 25.0 -> 22.2 mm
- net /PARPORT_PD7: track 26.3 -> 23.5 mm
- net /~{PARPORT_STB}: track 30.9 -> 28.1 mm
- net Net-(U2-RA2): track 18.8 -> 16.0 mm
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Other:
- board size 108.3 x 89.9 mm -> 107.3 x 89.9 mm
- board text added: "Go LPT It Out 2025-04-23 by rglenn"
- board text removed: "Go LPT It Out 2025-01-05 by rglenn"
