File: go-lpt-it-out/go-lpt-it-out.kicad_sch (KiCad schematic)
At the start: 19 parts, among them J1 Bus_ISA_8bit, J2 DE9, J3 Parallel, J4 Conn_02x05_Odd_Even, Q1 MMBT3904, U1 TL16C552A, U2 GD75232N, U3 GD75232N, U6 74HCU04, Y1 1.8432MHz

Commit message: Adding updates to go-lpt-it-out
Parts:
- J2: footprint Connector_Dsub:DSUB-9_Male_Horizontal_P2.77x2.84mm_EdgePinOffset4.94mm_Housed_MountingHolesOffset4.94mm -> Connector_Dsub:DSUB-9_Pins_Horizontal_P2.77x2.84mm_EdgePinOffset7.70mm_Housed_MountingHolesOffset9.12mm
- J3: footprint Connector_Dsub:DSUB-25_Female_Horizontal_P2.77x2.84mm_EdgePinOffset4.94mm_Housed_MountingHolesOffset4.94mm -> Connector_Dsub:DSUB-25_Socket_Horizontal_P2.77x2.84mm_EdgePinOffset7.70mm_Housed_MountingHolesOffset9.12mm
