File: rom-n-roll-star/rom-n-roll-star.kicad_pcb (KiCad board)
At the start: 2 copper layers, 104.5 x 74.9 mm, 16 parts, among them J1 Bus_ISA_8bit, SW1 SW_DIP_x08, U1 SST39SF010, U2 74ALS688

Commit message: Adding last-minute changes to rom-n-roll-star
Other:
- board size 104.5 x 74.9 mm -> 103.5 x 74.9 mm
