File: the-importance-of-being-ide/the-importance-of-being-ide.kicad_pcb (KiCad board)
At the start: 4 copper layers, 165.4 x 88.9 mm, 71 parts, among them J1 Bus_ISA_16bit, J2 Conn_02x20_Odd_Even, J3 Conn_02x20_Odd_Even, J4 IDE1_ACT, J5 IDE2_ACT, J6 IDE_ACT, SW1 SW_DIP_x08, U1 SST39SF010, U10 74ALS125, U11 74ALS125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

Commit message: Adding last minute changes to the-importance-of-being-ide
Routing:
- net /AEN: track 107.7 -> 107.1 mm
Other:
- board size 165.4 x 88.9 mm -> 164.4 x 88.9 mm
