File: usb-in-the-sky/usb-in-the-sky.kicad_pcb (KiCad board)
At the start: 2 copper layers, 107.6 x 73 mm, 28 parts, among them J1 Bus_ISA_8bit, J2 USB_A, SW1 SW_DIP_x05, U1 CH375, U2 74LS688, U3 74LS245, U4 74ALS688, U5 SST39SF010, U6 USBLC6-2SC6, Y1 12 MHz

Commit message: Adding latest updates to usb-in-the-sky
Parts:
- BRACKET1: footprint pc-parts:PC_BRACKET_ISA_KEYSTONE_9200_Rev1_1 -> pc-parts:PC_BRACKET_ISA_KEYSTONE_9202_Rev1
Other:
- board size 107.6 x 73 mm -> 106.6 x 73 mm
- board text added: "USB In The Sky 2025-01-05 by rglenn"
