File: dont-look-backplane-in-anger-2/isa_backplane.kicad_sch (KiCad schematic)
At the start: 121 parts, among them J1 MINUS5, P1 POWER_SW, P2 RESET, P3 POWER, P4 SERIAL, P5 SERIAL, P6 RESET, P7 POWER_LED, Q1 2N3906, Q2 2N3906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

Commit message: Updating footprint and 3D model for ISA slots
Parts:
- BUS1, BUS2, BUS3, BUS4, BUS5, BUS6, BUS7, BUS8: footprint (none) -> pc-parts:645169-3
Changed lines of the file:
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@@
 			)
 		)
-		(property "Footprint" ""
+		(property "Footprint" "pc-parts:645169-3"
 			(at 55.88 90.17 0)
 			(effects
@@
 			)
 		)
-		(property "Footprint" ""
+		(property "Footprint" "pc-parts:645169-3"
 			(at 137.16 90.17 0)
 			(effects
@@
 			)
 		)
-		(property "Footprint" ""
+		(property "Footprint" "pc-parts:645169-3"
 			(at 218.44 90.17 0)
 			(effects
@@
 			)
 		)
-		(property "Footprint" ""
+		(property "Footprint" "pc-parts:645169-3"
 			(at 299.72 90.17 0)
 			(effects
@@
 			)
 		)
-		(property "Footprint" ""
+		(property "Footprint" "pc-parts:645169-3"
 			(at 55.88 227.33 0)
 			(effects
@@
 			)
 		)
-		(property "Footprint" ""
+		(property "Footprint" "pc-parts:645169-3"
 			(at 137.16 227.33 0)
 			(effects
@@
 			)
 		)
-		(property "Footprint" ""
+		(property "Footprint" "pc-parts:645169-3"
 			(at 299.72 226.06 0)
 			(effects
@@
 			)
 		)
-		(property "Footprint" ""
+		(property "Footprint" "pc-parts:645169-3"
 			(at 218.44 226.06 0)
 			(effects
